Commit message: ports

File: src/cra_description/urdf/cr10_robot.xacro (robot description, xacro)
@@ -508,7 +508,9 @@
     </hardware>
     <joint name="joint1">
-      <command_interface name="position">
-        <param name="min">-1</param><param name="max">1</param>
-      </command_interface>
+      <!-- min/max removidos: eram placeholders ±1 rad do fork Dobot e
+           CLAMPAVAM o comando — joint3 (home −2,094) e joint5 (home
+           +1,571) ficam fora de [−1,1]. Sem os params, o gazebo_ros2_control
+           usa os <limit> reais da junta (±6,27; joint3 ±2,861). -->
+      <command_interface name="position"/>
       <state_interface name="position">
         <param name="initial_value">-0.7854</param>
@@ -517,7 +519,9 @@
     </joint>
     <joint name="joint2">
-      <command_interface name="position">
-        <param name="min">-1</param><param name="max">1</param>
-      </command_interface>
+      <!-- min/max removidos: eram placeholders ±1 rad do fork Dobot e
+           CLAMPAVAM o comando — joint3 (home −2,094) e joint5 (home
+           +1,571) ficam fora de [−1,1]. Sem os params, o gazebo_ros2_control
+           usa os <limit> reais da junta (±6,27; joint3 ±2,861). -->
+      <command_interface name="position"/>
       <state_interface name="position">
         <param name="initial_value">0.5236</param>
@@ -526,7 +530,9 @@
     </joint>
     <joint name="joint3">
-      <command_interface name="position">
-        <param name="min">-1</param><param name="max">1</param>
-      </command_interface>
+      <!-- min/max removidos: eram placeholders ±1 rad do fork Dobot e
+           CLAMPAVAM o comando — joint3 (home −2,094) e joint5 (home
+           +1,571) ficam fora de [−1,1]. Sem os params, o gazebo_ros2_control
+           usa os <limit> reais da junta (±6,27; joint3 ±2,861). -->
+      <command_interface name="position"/>
       <state_interface name="position">
         <param name="initial_value">-2.0944</param>
@@ -535,7 +541,9 @@
     </joint>
     <joint name="joint4">
-      <command_interface name="position">
-        <param name="min">-1</param><param name="max">1</param>
-      </command_interface>
+      <!-- min/max removidos: eram placeholders ±1 rad do fork Dobot e
+           CLAMPAVAM o comando — joint3 (home −2,094) e joint5 (home
+           +1,571) ficam fora de [−1,1]. Sem os params, o gazebo_ros2_control
+           usa os <limit> reais da junta (±6,27; joint3 ±2,861). -->
+      <command_interface name="position"/>
       <state_interface name="position">
         <param name="initial_value">0.0</param>
@@ -544,7 +552,9 @@
     </joint>
     <joint name="joint5">
-      <command_interface name="position">
-        <param name="min">-1</param><param name="max">1</param>
-      </command_interface>
+      <!-- min/max removidos: eram placeholders ±1 rad do fork Dobot e
+           CLAMPAVAM o comando — joint3 (home −2,094) e joint5 (home
+           +1,571) ficam fora de [−1,1]. Sem os params, o gazebo_ros2_control
+           usa os <limit> reais da junta (±6,27; joint3 ±2,861). -->
+      <command_interface name="position"/>
       <state_interface name="position">
         <param name="initial_value">1.5708</param>
@@ -553,7 +563,9 @@
     </joint>
     <joint name="joint6">
-      <command_interface name="position">
-        <param name="min">-1</param><param name="max">1</param>
-      </command_interface>
+      <!-- min/max removidos: eram placeholders ±1 rad do fork Dobot e
+           CLAMPAVAM o comando — joint3 (home −2,094) e joint5 (home
+           +1,571) ficam fora de [−1,1]. Sem os params, o gazebo_ros2_control
+           usa os <limit> reais da junta (±6,27; joint3 ±2,861). -->
+      <command_interface name="position"/>
       <state_interface name="position">
         <param name="initial_value">0.0</param>
