Commit message: celula de carga antiga

File: src/touch_pack/urdf/touch_tool_tcp.urdf (robot description, URDF)
Before this commit: robot touch_tool_tcp, 7 links, 6 joints
Links:
- removed link ft_flange_link
- removed link ft_sensor_link
- added link coupler_robot_link, mass 0.0419; collision cylinder length=0.0185 radius=0.03175; visual mesh filename=package://touch_pack/meshes/acoplador_robo.stl scale=0.001 0.001 0.001
- added link load_cell_link, mass 0.4748; collision box size=0.0508 0.0191 0.0702; visual mesh filename=package://touch_pack/meshes/celula_carga_100kg.stl scale=0.001 0.001 0.001
- added link touch_tool_link, mass 0.0366; collision cylinder length=0.046 radius=0.029; visual mesh filename=package://touch_pack/meshes/touch_tool.stl scale=0.001 0.001 0.001
- link coupler_tool_link: mass 0.0275 -> 0.0444; geometry collision cylinder length=0.013 radius=0.03175; visual mesh filename=package://touch_pack/meshes/acoplador_tool.stl scale=0.001 0.001 0.001
- link tool_tip_link: mass 0.0043 -> 0.0057; geometry collision box size=0.0170 0.0195 0.0005; collision box size=0.0224 0.0249 0.004
Joints:
- removed joint ft_flange_attach
- removed joint ft_sensor_attach
- removed joint tool_tip_sleeve_attach
- added joint coupler_robot_attach: type fixed, parent Link6, child coupler_robot_link, origin xyz=0 0 0 rpy=0 0 0
- added joint load_cell_attach: type fixed, parent coupler_robot_link, child load_cell_link, origin xyz=0 0 0.0155 rpy=0 0 0
- added joint tool_tip_attach: type fixed, parent touch_tool_link, child tool_tip_link, origin xyz=0 0 0.046 rpy=0 0 0
- added joint touch_tool_attach: type fixed, parent coupler_tool_link, child touch_tool_link, origin xyz=0 0 0.013 rpy=0 0 0
- joint coupler_tool_attach: origin xyz=0 0 0.0368 rpy=0 0 0 -> xyz=0 0 0.0732 rpy=0 0 0; parent ft_sensor_link -> load_cell_link
- joint tcp_alias_joint: origin xyz=0 0 0.018 rpy=0 0 0 -> xyz=0 0 0.0145 rpy=0 0 0

Commit message: new load cell ft6

File: src/touch_pack/urdf/touch_tool_tcp.urdf (robot description, URDF)
Before this commit: robot touch_tool_tcp, 8 links, 7 joints
Links:
- removed link coupler_robot_link
- removed link touch_tool_link
- added link ft_flange_link, mass 0.0518; collision cylinder length=0.006 radius=0.0375; visual mesh filename=package://touch_pack/meshes/fa7155_flange_fixo.stl scale=0.001 0.001 0.001
- link coupler_tool_link: mass 0.0444 -> 0.0275; geometry collision cylinder length=0.0025 radius=0.0075; collision cylinder length=0.010 radius=0.033
- link load_cell_link: mass 0.4748 -> 0.3000; geometry collision cylinder length=0.0309 radius=0.0375; visual mesh filename=package://touch_pack/meshes/fa7155_sensor.stl scale=0.001 0.001 0.001
- link tool_tip_link: mass 0.0057 -> 0.0043; geometry collision box size=0.0150 0.0170 0.0020; collision box size=0.020 0.020 0.016
Joints:
- removed joint coupler_robot_attach
- removed joint touch_tool_attach
- added joint ft_flange_attach: type fixed, parent Link6, child ft_flange_link, origin xyz=0 0 0 rpy=0 0 0
- joint coupler_tool_attach: origin xyz=0 0 0.0732 rpy=0 0 0 -> xyz=0 0 0.0368 rpy=0 0 0
- joint load_cell_attach: origin xyz=0 0 0.0155 rpy=0 0 0 -> xyz=0 0 0.0004 rpy=0 0 0; parent coupler_robot_link -> ft_flange_link
- joint tcp_alias_joint: origin xyz=0 0 0.0145 rpy=0 0 0 -> xyz=0 0 0.018 rpy=0 0 0
- joint tool_tip_attach: origin xyz=0 0 0.046 rpy=0 0 0 -> xyz=0 0 0.0125 rpy=0 0 0; parent touch_tool_link -> coupler_tool_link
